Commit message: [jsk_spot_startup] add respeaker_base to xacro

File: jsk_spot_robot/jsk_spot_startup/robots/insta_360_air_mount.urdf.xacro (robot description, xacro)
@@ -7,3 +7,9 @@
         <child link="camera" />
     </joint>
+    <link name="respeaker_base" />
+    <joint name="head_mount_to_respeaker_base" type="fixed">
+        <origin rpy="0 0 0" xyz="0 0 0.05" />
+        <parent_link="jsk_head_mount_frame" />
+        <child link="respeaker_base" />
+    </joint>
 </robot>

Commit message: [jsk_spot_startup] fix typo in xacro

File: jsk_spot_robot/jsk_spot_startup/robots/insta_360_air_mount.urdf.xacro (robot description, xacro)
@@ -10,5 +10,5 @@
     <joint name="head_mount_to_respeaker_base" type="fixed">
         <origin rpy="0 0 0" xyz="0 0 0.05" />
-        <parent_link="jsk_head_mount_frame" />
+        <parent link="jsk_head_mount_frame" />
         <child link="respeaker_base" />
     </joint>
