Commit message: [jsk_fetch_startup] update jsk fetch models

File: jsk_fetch_robot/jsk_fetch_startup/robots/head_l515.urdf.xacro (robot description, xacro)
@@ -23,8 +23,14 @@
     </collision>
   </link>
-  <joint name="head_l515_mount_virtual_joint" type="fixed">
+  <joint name="head_l515_mount_link_virtual_joint" type="fixed">
+    <origin rpy="1.57 0 -1.57" xyz="0.02 0.05 0.0" />
+    <parent link="head_l515_virtual_mount_link" />
+    <child link="head_l515_mount_link" />
+  </joint>
+  <link name="head_l515_virtual_mount_link" />
+  <joint name="head_l515_virtual_mount_link_virtual_joint" type="fixed">
     <origin rpy="0 0 0" xyz="0.0255 0 0.055" />
     <parent link="head_tilt_link" />
-    <child link="head_l515_mount_link" />
+    <child link="head_l515_virtual_mount_link" />
   </joint>
   <link name="l515_head_link"/>

File: jsk_fetch_robot/jsk_fetch_startup/robots/jsk_fetch.urdf.xacro (robot description, xacro)
@@ -2,8 +2,9 @@
 <robot name="fetch" xmlns:xacro="http://www.ros.org/wiki/xacro">
   <xacro:arg name="ros_distro" default="melodic" />
+  <xacro:arg name="use_fetch_description" default="false" />
   <xacro:arg name="base_camera_mount" default="true" />
-  <xacro:arg name="head_box" default="true" />
+  <xacro:arg name="head_box" default="false" />
   <xacro:arg name="head_l515" default="true" />
-  <xacro:arg name="use_fetch_description" default="false" />
+  <xacro:arg name="insta360_stand" default="true" />
   <xacro:if value="$(arg use_fetch_description)">
     <xacro:include filename="$(find fetch_description)/robots/fetch.urdf" />
@@ -21,3 +22,6 @@
     <xacro:include filename="$(find jsk_fetch_startup)/robots/head_l515.urdf.xacro" />
   </xacro:if>
+  <xacro:if value="$(arg insta360_stand)">
+    <xacro:include filename="$(find jsk_fetch_startup)/robots/insta360_stand.urdf.xacro" />
+  </xacro:if>
 </robot>
